File: ADAP030/ADAP030.brd (EAGLE design)
At the start: 86.7 x 43.5 mm, 19 parts, among them IC1 68020, IC2 68030, IC3 GAL22V10

Commit message: CBACK
Parts:
- moved R6 0.32 mm to (74.3, 2.86), turned to 0 degrees
Routing:
- net VCC: track 53.3 -> 64.7 mm
- net CBACK: track 0.00 -> 5.74 mm
- net SIZ1: track 47.8 -> 49.2 mm
Other:
- board text added: "v1.1"
Changed lines of the file:
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@@
 <layer number="20" name="Dimension" color="15" fill="1" visible="yes" active="yes"/>
 <layer number="21" name="tPlace" color="7" fill="1" visible="yes" active="yes"/>
-<layer number="22" name="bPlace" color="7" fill="1" visible="no" active="yes"/>
+<layer number="22" name="bPlace" color="7" fill="1" visible="yes" active="yes"/>
 <layer number="23" name="tOrigins" color="15" fill="1" visible="yes" active="yes"/>
 <layer number="24" name="bOrigins" color="15" fill="1" visible="no" active="yes"/>
-<layer number="25" name="tNames" color="7" fill="1" visible="no" active="yes"/>
+<layer number="25" name="tNames" color="7" fill="1" visible="yes" active="yes"/>
 <layer number="26" name="bNames" color="7" fill="1" visible="no" active="yes"/>
 <layer number="27" name="tValues" color="7" fill="1" visible="no" active="yes"/>
@@
 <text x="85.4075" y="0.9525" size="1.4224" layer="1" font="vector" rot="R90">Top</text>
 <text x="84.455" y="40.64" size="1.4224" layer="16" font="vector" rot="MR0">Bottom</text>
+<text x="27.6225" y="42.8625" size="1.4224" layer="1" font="vector" rot="R180">v1.1</text>
+<text x="24.765" y="27.6225" size="1.4224" layer="25" font="vector" rot="R270">v1.1</text>
 </plain>
 <attributes>
@@
 <attribute name="OC_FARNELL" value="unknown" x="67.6275" y="22.225" size="1.778" layer="27" rot="R90" display="off"/>
 <attribute name="OC_NEWARK" value="52F3269" x="67.6275" y="22.225" size="1.778" layer="27" rot="R90" display="off"/>
-<attribute name="NAME" x="69.85" y="4.1275" size="1.778" layer="25" ratio="10" rot="R180"/>
+<attribute name="NAME" x="59.055" y="3.81" size="1.778" layer="25" ratio="10" rot="R180"/>
 <attribute name="VALUE" x="71.755" y="18.7325" size="1.778" layer="27" ratio="10" rot="R180"/>
 </element>
@@
 <attribute name="VALUE" x="5.55" y="6.095" size="1.016" layer="28" rot="MR180"/>
 </element>
-<element name="R6" library="rcl" package="M0805" value="10k" x="74.295" y="3.175" rot="R180"/>
+<element name="R6" library="rcl" package="M0805" value="10k" x="74.295" y="2.8575" smashed="yes">
+<attribute name="NAME" x="69.7865" y="1.016" size="1.27" layer="25"/>
+<attribute name="VALUE" x="73.279" y="0.5715" size="1.27" layer="27"/>
+</element>
 </elements>
 <signals>
@@
 <wire x1="75.8825" y1="19.685" x2="77.7875" y2="19.685" width="0.2" layer="16"/>
 <contactref element="R6" pad="1"/>
-<wire x1="70.1675" y1="12.065" x2="75.245" y2="3.175" width="0" layer="19" extent="1-1"/>
+<wire x1="70.1675" y1="12.065" x2="71.12" y2="11.1125" width="0.15" layer="1"/>
+<wire x1="71.12" y1="11.1125" x2="71.12" y2="3.4925" width="0.15" layer="1"/>
+<wire x1="71.12" y1="3.4925" x2="71.755" y2="2.8575" width="0.15" layer="1"/>
+<wire x1="71.755" y1="2.8575" x2="73.345" y2="2.8575" width="0.15" layer="1"/>
 </signal>
 <signal name="/RESET">
@@
 <wire x1="40.9575" y1="6.985" x2="40.9575" y2="5.08" width="0.15" layer="16"/>
 <wire x1="40.9575" y1="5.08" x2="41.5925" y2="4.445" width="0.15" layer="16"/>
-<wire x1="41.5925" y1="4.445" x2="70.8025" y2="4.445" width="0.15" layer="16"/>
-<wire x1="70.8025" y1="4.445" x2="71.4375" y2="3.81" width="0.15" layer="16"/>
-<via x="71.4375" y="3.81" extent="1-16" drill="0.3"/>
-<wire x1="71.4375" y1="3.81" x2="71.4375" y2="8.255" width="0.15" layer="1"/>
-<wire x1="71.4375" y1="8.255" x2="72.7075" y2="9.525" width="0.15" layer="1"/>
+<wire x1="41.5925" y1="4.445" x2="71.12" y2="4.445" width="0.15" layer="16"/>
+<wire x1="71.12" y1="4.445" x2="71.755" y2="3.81" width="0.15" layer="16"/>
+<via x="71.755" y="3.81" extent="1-16" drill="0.3"/>
+<wire x1="71.755" y1="3.81" x2="71.755" y2="8.5725" width="0.15" layer="1"/>
+<wire x1="71.755" y1="8.5725" x2="72.7075" y2="9.525" width="0.15" layer="1"/>
 </signal>
 <signal name="/IPL1">
@@
 <wire x1="41.91" y1="10.4775" x2="41.91" y2="5.3975" width="0.15" layer="16"/>
 <wire x1="41.91" y1="5.3975" x2="42.545" y2="4.7625" width="0.15" layer="16"/>
-<wire x1="42.545" y1="4.7625" x2="72.0725" y2="4.7625" width="0.15" layer="16"/>
-<wire x1="72.0725" y1="4.7625" x2="72.39" y2="4.445" width="0.15" layer="16"/>
-<wire x1="72.39" y1="4.445" x2="82.8675" y2="4.445" width="0.15" layer="16"/>
+<wire x1="42.545" y1="4.7625" x2="74.6125" y2="4.7625" width="0.15" layer="16"/>
+<wire x1="74.6125" y1="4.7625" x2="74.93" y2="4.445" width="0.15" layer="16"/>
+<wire x1="74.93" y1="4.445" x2="82.8675" y2="4.445" width="0.15" layer="16"/>
 <via x="82.8675" y="4.445" extent="1-16" drill="0.3"/>
 <wire x1="82.8675" y1="4.445" x2="83.82" y2="5.3975" width="0.15" layer="1"/>
@@
 <wire x1="56.1975" y1="10.16" x2="56.515" y2="10.4775" width="0.15" layer="1"/>
 <wire x1="56.515" y1="10.4775" x2="56.8325" y2="10.4775" width="0.15" layer="1"/>
-<wire x1="74.295" y1="11.1125" x2="75.2475" y2="12.065" width="0.15" layer="1"/>
 <wire x1="56.8325" y1="10.4775" x2="57.4675" y2="11.1125" width="0.15" layer="1"/>
-<wire x1="57.4675" y1="11.1125" x2="74.295" y2="11.1125" width="0.15" layer="1"/>
+<wire x1="57.4675" y1="11.1125" x2="68.2625" y2="11.1125" width="0.15" layer="1"/>
+<wire x1="68.2625" y1="11.1125" x2="68.8975" y2="11.7475" width="0.15" layer="1"/>
+<wire x1="68.8975" y1="11.7475" x2="68.8975" y2="12.7" width="0.15" layer="1"/>
+<wire x1="68.8975" y1="12.7" x2="69.215" y2="13.0175" width="0.15" layer="1"/>
+<wire x1="69.215" y1="13.0175" x2="74.295" y2="13.0175" width="0.15" layer="1"/>
+<wire x1="74.295" y1="13.0175" x2="75.2475" y2="12.065" width="0.15" layer="1"/>
 </signal>
 <signal name="/RMC">
@@
 <wire x1="43.4975" y1="6.985" x2="43.4975" y2="5.715" width="0.15" layer="16"/>
 <wire x1="43.4975" y1="5.715" x2="44.1325" y2="5.08" width="0.15" layer="16"/>
-<wire x1="44.1325" y1="5.08" x2="75.2475" y2="5.08" width="0.15" layer="16"/>
-<via x="75.2475" y="5.08" extent="1-16" drill="0.3"/>
-<wire x1="75.2475" y1="5.08" x2="76.2" y2="6.0325" width="0.15" layer="1"/>
-<wire x1="76.2" y1="6.0325" x2="76.2" y2="8.5725" width="0.15" layer="1"/>
+<wire x1="44.1325" y1="5.08" x2="75.565" y2="5.08" width="0.15" layer="16"/>
+<via x="75.565" y="5.08" extent="1-16" drill="0.3"/>
+<wire x1="75.565" y1="5.08" x2="76.2" y2="5.715" width="0.15" layer="1"/>
+<wire x1="76.2" y1="5.715" x2="76.2" y2="8.5725" width="0.15" layer="1"/>
 <wire x1="76.2" y1="8.5725" x2="75.2475" y2="9.525" width="0.15" layer="1"/>
 </signal>
@@
 <contactref element="R6" pad="2"/>
 <contactref element="IC2" pad="J01"/>
-<wire x1="73.345" y1="3.175" x2="72.7075" y2="6.985" width="0" layer="19" extent="1-1"/>
+<wire x1="72.7075" y1="6.985" x2="72.7075" y2="5.715" width="0.15" layer="1"/>
+<wire x1="72.7075" y1="5.715" x2="73.3425" y2="5.08" width="0.15" layer="1"/>
+<wire x1="73.3425" y1="5.08" x2="74.295" y2="5.08" width="0.15" layer="1"/>
+<wire x1="74.295" y1="5.08" x2="75.2475" y2="4.1275" width="0.15" layer="1"/>
+<wire x1="75.2475" y1="4.1275" x2="75.2475" y2="2.86" width="0.15" layer="1"/>
+<wire x1="75.2475" y1="2.86" x2="75.245" y2="2.8575" width="0.15" layer="1"/>
 </signal>
 </signals>
