File: ADAP030/ADAP030.sch (EAGLE design)
At the start: 19 parts, among them IC1 68020, IC2 68030, IC3 GAL22V10

Commit message: CBACK
Changed lines of the file:
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@@
 <pinref part="IC2" gate="G$1" pin="IPEND"/>
 <wire x1="205.74" y1="116.84" x2="185.42" y2="116.84" width="0.1524" layer="91"/>
+<label x="185.42" y="116.84" size="1.778" layer="95"/>
 </segment>
 </net>
